Commit message: till map

File: src/simple_rover_description/urdf/simple_rover.urdf.xacro (robot description, xacro)
@@ -4,8 +4,8 @@
   <link name="left_wheel"/>
   <link name="right_wheel"/>
-  <link name="lidar_link"/>
-  <joint name="lidar_joint" type="fixed">
+  <link name="laser"/>
+  <joint name="laser_joint" type="fixed">
     <parent link="base_link"/>
-    <child link="lidar_link"/>
+    <child link="laser"/>
     <origin xyz="0.12 0 0.12" rpy="0 0 0"/>
   </joint>

File: urdf/your_robot.urdf (robot description, URDF)
Before this commit: robot simple_rover, 2 links, 1 joints
Links:
- link laser: mass 0.1 -> None
Joints:
- joint laser_joint: origin xyz=0.12 0 0.25 rpy=0 0 0 -> xyz=0.12 0 0.12 rpy=0 0 0

Commit message: working dynamic tf

File: src/simple_rover_description/urdf/simple_rover.urdf.xacro (robot description, xacro)
@@ -8,5 +8,5 @@
     <parent link="base_link"/>
     <child link="laser"/>
-    <origin xyz="0.12 0 0.12" rpy="0 0 0"/>
+    <origin xyz="0.2 0 0.15" rpy="0 0 0"/>
   </joint>
   <!-- wheel joints are fixed in this simple model (no visuals needed) -->

Commit message: map works

File: src/simple_rover_description/urdf/simple_rover.urdf.xacro (robot description, xacro)
@@ -4,8 +4,8 @@
   <link name="left_wheel"/>
   <link name="right_wheel"/>
-  <link name="laser"/>
+  <link name="laser_frame"/>
   <joint name="laser_joint" type="fixed">
     <parent link="base_link"/>
-    <child link="laser"/>
+    <child link="laser_frame"/>
     <origin xyz="0.2 0 0.15" rpy="0 0 0"/>
   </joint>

Commit message: working till cmd-vel 0

File: src/simple_rover_description/urdf/simple_rover.urdf.xacro (robot description, xacro)
@@ -1,8 +1,34 @@
 <?xml version="1.0"?>
 <robot xmlns:xacro="http://www.ros.org/wiki/xacro" name="simple_rover">
-  <link name="base_link"/>
+  <!-- Ground reference -->
+  <link name="base_footprint"/>
+  <!-- Robot body -->
+  <link name="base_link">
+    <visual>
+      <geometry>
+        <box size="0.4 0.3 0.15"/>
+      </geometry>
+      <origin xyz="0 0 0.075"/>
+      <material name="gray"/>
+    </visual>
+  </link>
+  <!-- Laser -->
+  <link name="laser_frame">
+    <visual>
+      <geometry>
+        <cylinder radius="0.03" length="0.05"/>
+      </geometry>
+    </visual>
+  </link>
+  <!-- Wheels -->
   <link name="left_wheel"/>
   <link name="right_wheel"/>
-  <link name="laser_frame"/>
+  <!-- base_footprint → base_link -->
+  <joint name="base_footprint_to_base_link" type="fixed">
+    <parent link="base_footprint"/>
+    <child link="base_link"/>
+    <origin xyz="0 0 0" rpy="0 0 0"/>
+  </joint>
+  <!-- base_link → laser -->
   <joint name="laser_joint" type="fixed">
     <parent link="base_link"/>
@@ -10,14 +36,14 @@
     <origin xyz="0.2 0 0.15" rpy="0 0 0"/>
   </joint>
-  <!-- wheel joints are fixed in this simple model (no visuals needed) -->
+  <!-- Wheels -->
   <joint name="left_wheel_joint" type="fixed">
     <parent link="base_link"/>
     <child link="left_wheel"/>
-    <origin xyz="0 0.12 0" rpy="0 0 0"/>
+    <origin xyz="0 0.12 0"/>
   </joint>
   <joint name="right_wheel_joint" type="fixed">
     <parent link="base_link"/>
     <child link="right_wheel"/>
-    <origin xyz="0 -0.12 0" rpy="0 0 0"/>
+    <origin xyz="0 -0.12 0"/>
   </joint>
 </robot>
