Commit message: cmd to vel

File: urdf/your_robot.urdf (robot description, URDF)
Before this commit: robot simple_rover, 2 links, 1 joints
Links:
- removed link laser
- added link laser_frame
Joints:
- joint laser_joint: child laser -> laser_frame; origin xyz=0.12 0 0.12 rpy=0 0 0 -> xyz=0.20 0 0.20 rpy=0 0 0

Commit message: working cmd_vel 1

File: urdf/your_robot.urdf (robot description, URDF)
Before this commit: robot simple_rover, 2 links, 1 joints
Links:
- added link base_footprint, mass 0.1
Joints:
- added joint base_footprint_to_base_link: type fixed, parent base_footprint, child base_link, origin xyz=0 0 0 rpy=0 0 0
